Commit message: simulation improvements

File: src/pkg/rover_description_pkg/urdf/rover_macro.xacro (robot description, xacro)
@@ -49,5 +49,5 @@
                 <origin xyz="0.0 0.0 ${collision_z_elev}" rpy="0.0 0.0 0.0"/>
                 <geometry>
-                    <box size="${total_length} ${total_width - 2*track_width} ${total_height - 0.0005}"/>
+                    <box size="${total_length} ${total_width - 2*track_width} ${total_height - 0.1}"/>
                 </geometry>
             </collision>
@@ -69,10 +69,10 @@
             </geometry>
         </visual> -->
-        <collision>
-            <origin xyz="0 0.0115 0.05" rpy="0 0 0" />
+        <!-- <collision>
+            <origin xyz="-0.1 0.0 0.04" rpy="0 0 0" />
             <geometry>
-                <box size="${total_length} ${total_width -2*track_width} 0.03"/>
+                <box size="${total_length/3} ${total_width -4.5*track_width} 0.05"/>
             </geometry>
-        </collision>
+        </collision> -->
         <inertial>
             <origin xyz="-0.01 0 0" rpy="0 0 0"/>
@@ -95,9 +95,9 @@
             <parent link="payload_link"/>
             <child link="${laser_frame}"/>
-            <origin xyz="0.07 0 0.11" rpy="0 0 3.1415"/>
+            <origin xyz="0.075 0 0.04" rpy="0 3.1415 0"/>
         </joint>
         <link name="${laser_frame}">
             <visual>
-                <origin xyz="0 0 0" rpy="-1.57 0 3.1415"/>
+                <origin xyz="0 0 0" rpy="-1.57 3.1415 3.1415"/>
                 <geometry>
                     <mesh filename="file://$(find rover_description_pkg)/meshes/rplidar_s2.dae"/>
@@ -107,5 +107,5 @@
                 <origin xyz="0 0 -0.05" rpy="0 0 3.1415"/>
                 <geometry>
-                    <cylinder radius="0.05" length="0.15"/>
+                    <cylinder radius="0.04" length="0.15"/>
                 </geometry>
             </collision>
@@ -133,5 +133,5 @@
                 </scan>
                 <range>
-                <min>0.15</min>
+                <min>0.23</min>
                 <max>10.0</max>
                 <resolution>0.01</resolution>
