Commit message: urdf updated, dockerfile for drones simulation created, folder cleanse

File: src/pkg/rover_description_pkg/urdf/rover_macro.xacro (robot description, xacro)
@@ -1,5 +1,5 @@
 <?xml version="1.0"?>
 <robot xmlns:xacro="http://www.ros.org/wiki/xacro" name="rover_macro">
-    <!-- rover properties -->
+        <!-- rover properties -->
     <xacro:property name="track_width" value="0.08"/>
     <xacro:property name="total_width" value="0.4515"/>
@@ -11,13 +11,20 @@
     <xacro:property name="track_distance" value="0.2915"/>
     <xacro:property name="wheel_axes_distance" value="0.220"/>
-    <!-- this elevates the rover visuals and the collision boxes in order to make it above the ground floor
-        and make the collision boxes inglobate the rover visuals -->
-    <xacro:property name="rover_z_elev" value="${total_height/2 - chassis_height/2}"/>
-    <xacro:property name="collision_z_elev" value="${chassis_height/2}"/>
-    <!-- to have a collision box where the front and back tracks are, while in the middle there is the cylinder
-    that acts as a differential drive robot wheel -->
     <xacro:property name="wheel_collision_x" value="${total_length/2 - total_height/2 - 0.001}"/>
     <xacro:property name="wheel_collision_y" value="${track_width}"/>
     <xacro:property name="wheel_collision_z" value="${total_height - 0.02}"/>
+    <xacro:property name="rover_z_elev" value="${total_height/2 - chassis_height/2}"/>
+    <xacro:property name="collision_z_elev" value="${chassis_height/2}"/>
+    <!-- Robot Parameters -->
+    <xacro:property name="wheel_z_offset" value="0.020" />
+    <xacro:property name="wheel_x_offset" value="${wheel_axes_distance/2}" /> <!-- <xacro:property name="wheel_x_offset" value="0.145" /> -->
+    <xacro:property name="front_flipper_x_offset" value="-0.0035" />
+    <xacro:property name="wheel_y_offset" value="${(total_width-track_width)/2}" /> <!-- <xacro:property name="wheel_y_offset" value="0.18" /> -->
+    <xacro:property name="track_y_offset" value="0.11" />
+    <xacro:property name="wheel_mass" value="1.25" />
+    <xacro:property name="payload_z_offset" value="0.096" />
+    <!-- <xacro:include filename="$(find rover_description_pkg)/urdf/rover_dev_payload.urdf" />
+    <xacro:include filename="$(find rover_description_pkg)/urdf/rplidar_s2.urdf" /> -->
+    <xacro:include filename="$(find rover_description_pkg)/urdf/imu.urdf" />
     <xacro:macro name="rover_base_frame" params="parent_link">
         <joint name="world_base_joint" type="fixed">
@@ -28,8 +35,7 @@
         <link name="base_link">
             <visual>
-                <origin xyz="0.0 0.0 0.0" rpy="${PI/2} 0.0 ${PI/2}"/>
+                <origin xyz="0 0 -0.035" rpy="0 0 0" />
                 <geometry>
                     <mesh filename="file://$(find rover_description_pkg)/meshes/prisma_rover.dae" scale="0.001 0.001 0.001"/>
-                    <!--<mesh filename="package://rover_description_pkg/meshes/A4WD3-Tracked.stl" scale="0.001 0.001 0.001"/> -->
                 </geometry>
             </visual>
@@ -43,22 +49,101 @@
                 <origin xyz="0.0 0.0 ${collision_z_elev}" rpy="0.0 0.0 0.0"/>
                 <geometry>
-                    <box size="${total_length} ${total_width} ${total_height - 0.0005}"/>
+                    <box size="${total_length} ${total_width - 2*track_width} ${total_height - 0.0005}"/>
+                </geometry>
+            </collision>
+        </link>
+        <link name="pole_link">
+            <collision>
+            <origin xyz="0.0 0.0 0.0" rpy="0 0 0"/>
+                <geometry>
+                    <cylinder radius="0.0125" length="${1.1-2*total_height}"/>
                 </geometry>
             </collision>
         </link>
     </xacro:macro>
-    <xacro:macro name="rover_rplidar_s1" params="laser_frame">
-        <joint name="lidar_joint" type="fixed">
-            <parent link="base_footprint"/>
+    <link name="payload_link">
+        <!-- <visual>
+            <origin xyz="0 0.0115 0" rpy="1.57 -0 1.57" />
+            <geometry>
+                <mesh filename="file://$(find roverrobotics_description)/meshes/rover_payload.dae"/>
+            </geometry>
+        </visual> -->
+        <collision>
+            <origin xyz="0 0.0115 0.05" rpy="0 0 0" />
+            <geometry>
+                <box size="${total_length} ${total_width -2*track_width} 0.03"/>
+            </geometry>
+        </collision>
+        <inertial>
+            <origin xyz="-0.01 0 0" rpy="0 0 0"/>
+            <mass value="2.95" />
+            <inertia ixx="0.018398" ixy="0.0"  ixz="0.0" iyy="0.04064" iyz="0.0" izz="0.05396" />
+        </inertial>
+    </link>
+    <joint name="payload_to_base" type="fixed">
+        <parent link="base_link"/>
+        <child link="payload_link"/>
+        <origin xyz="0 0 ${payload_z_offset}"/>
+    </joint>
+    <joint name="pole_to_payload" type="fixed">
+        <origin xyz="0 0 ${ 0.5 - total_height/2}" rpy="0 0 0"/>
+        <parent link="payload_link"/>
+        <child link="pole_link"/>
+    </joint>
+<xacro:macro name="lidar_gazebo_sensor" params="laser_frame laser_topic">
+        <joint name="lidar_to_payload" type="fixed">
+            <parent link="payload_link"/>
             <child link="${laser_frame}"/>
-            <origin xyz="0.0 0.0 0.23" rpy="0.0 3.14 0 "/> <!-- RP_lidar has a 180 deg rotation on y and 0 on z -->
+            <origin xyz="0.07 0 0.11" rpy="0 0 3.1415"/>
         </joint>
         <link name="${laser_frame}">
-            <inertial>
-                <origin xyz="0.0 0.0 0.0" rpy="0.0 0.0 0.0"/>
-                <mass value="0.001"/>
-                <inertia ixx="0.001" ixy="0.0" ixz="0.0" iyy="0.001" iyz="0.0" izz="0.001"/>
-            </inertial>
+            <visual>
+                <origin xyz="0 0 0" rpy="-1.57 0 3.1415"/>
+                <geometry>
+                    <mesh filename="file://$(find rover_description_pkg)/meshes/rplidar_s2.dae"/>
+                </geometry>
+            </visual>
+            <collision>
+                <origin xyz="0 0 -0.05" rpy="0 0 3.1415"/>
+                <geometry>
+                    <cylinder radius="0.05" length="0.15"/>
+                </geometry>
+            </collision>
         </link>
+        <gazebo reference="${laser_frame}">
+        <sensor name='gpu_lidar' type='gpu_lidar'>
+            <pose>0 0 0 0 0 0</pose>
+            <topic>${laser_topic}</topic>
+            <ignition_frame_id>rover/lidar_link</ignition_frame_id>
+            <update_rate>10</update_rate>
+            <lidar>
+                <scan>
+                <horizontal>
+                    <samples>640</samples>
+                    <resolution>1</resolution>
+                    <min_angle>-3.14159</min_angle>
+                    <max_angle>3.14159</max_angle>
+                </horizontal>
+                <vertical>
+                    <samples>1</samples>
+                    <resolution>1</resolution>
+                    <min_angle>0.0</min_angle>
+                    <max_angle>0.0</max_angle>
+                </vertical>
+                </scan>
+                <range>
+                <min>0.15</min>
+                <max>10.0</max>
+                <resolution>0.01</resolution>
+                </range>
+            </lidar>
+            <visualize>true</visualize>
+        </sensor>
+    </gazebo>
+    <!-- <gazebo>
+        <plugin filename="libignition-gazebo-sensors-system.so" name="ignition::gazebo::systems::Sensors">
+            <render_engine>ogre2</render_engine>
+        </plugin>
+    </gazebo> -->
     </xacro:macro>
 <!--

Commit message: teleop node fpr remote control and new docker run init for fover inizialization

File: src/pkg/rover_description_pkg/urdf/rover.xacro (robot description, xacro)
@@ -14,5 +14,5 @@
     <xacro:gazebo_diff_drive_controller left_joint="diff_drive_l_joint" right_joint="diff_drive_r_joint"/>
     <xacro:gazebo_wheel_contact/>
-    <xacro:lidar_gazebo_sensor laser_frame="lidar_link" laser_topic="/scan"/>
+    <xacro:lidar_gazebo_sensor laser_frame="lidar_link" laser_topic="scan"/>
     <!-- <xacro:rover_payload_frame payload_frame="payload_link"/> -->
     <xacro:camera_gazebo camera_base_frame="camera_link" camera_topic="camera" camera_info_topic="camera_info"/>

File: src/pkg/rover_description_pkg/urdf/rover_gazebo.xacro (robot description, xacro)
@@ -115,5 +115,5 @@
     <!-- <xacro:sensor_d435i parent="${camera_base_frame}" use_nominal_extrinsics="true">
         <origin xyz="0 0 0" rpy="0 0 0"/>
-    </xacro:sensor_d435i> -->
+    </xacro:sensor_d435i>  -->
     <joint name="camera_to_payload" type="fixed">
         <origin xyz="0.02 0 ${1 -0.085 - total_height}" rpy="0 0 0"/>

File: src/pkg/rover_description_pkg/urdf/rover_macro.xacro (robot description, xacro)
@@ -95,9 +95,9 @@
             <parent link="payload_link"/>
             <child link="${laser_frame}"/>
-            <origin xyz="0.07 0 0.11" rpy="0 0 3.1415"/>
+            <origin xyz="0.075 0 0.035" rpy="0 3.1415 0.0"/>
         </joint>
         <link name="${laser_frame}">
             <visual>
-                <origin xyz="0 0 0" rpy="-1.57 0 3.1415"/>
+                <origin xyz="0 0 0" rpy="-1.57 3.1415 3.1415"/>
                 <geometry>
                     <mesh filename="file://$(find rover_description_pkg)/meshes/rplidar_s2.dae"/>
@@ -116,5 +116,5 @@
             <topic>${laser_topic}</topic>
             <ignition_frame_id>rover/lidar_link</ignition_frame_id>
-            <update_rate>10</update_rate>
+            <update_rate>30</update_rate>
             <lidar>
                 <scan>

Commit message: Dockerfile update and urdf adjustment

File: src/pkg/rover_description_pkg/urdf/rover.xacro (robot description, xacro)
@@ -15,5 +15,4 @@
     <xacro:gazebo_wheel_contact/>
     <xacro:lidar_gazebo_sensor laser_frame="lidar_link" laser_topic="scan"/>
-    <!-- <xacro:rover_payload_frame payload_frame="payload_link"/> -->
     <xacro:camera_gazebo camera_base_frame="camera_link" camera_topic="camera" camera_info_topic="camera_info"/>
 </xacro:if>

File: src/pkg/rover_description_pkg/urdf/rover_gazebo.xacro (robot description, xacro)
@@ -117,5 +117,5 @@
     </xacro:sensor_d435i>  -->
     <joint name="camera_to_payload" type="fixed">
-        <origin xyz="0.02 0 ${1 -0.085 - total_height}" rpy="0 0 0"/>
+        <origin xyz="0.02 0 ${1 -0.1 - total_height}" rpy="0 0 0"/>
         <parent link="payload_link"/>
         <child link="${camera_base_frame}"/>

File: src/pkg/rover_description_pkg/urdf/rover_macro.xacro (robot description, xacro)
@@ -69,10 +69,10 @@
             </geometry>
         </visual> -->
-        <!-- <collision>
+        <collision>
             <origin xyz="-0.1 0.0 0.04" rpy="0 0 0" />
             <geometry>
-                <box size="${total_length/3} ${total_width -4.5*track_width} 0.05"/>
+                <box size="${total_length/4} ${total_width -4.5*track_width} 0.04"/>
             </geometry>
-        </collision> -->
+        </collision>
         <inertial>
             <origin xyz="-0.01 0 0" rpy="0 0 0"/>
@@ -84,8 +84,8 @@
         <parent link="base_link"/>
         <child link="payload_link"/>
-        <origin xyz="0 0 ${payload_z_offset}"/>
+        <origin xyz="0 0 0.14"/>
     </joint>
     <joint name="pole_to_payload" type="fixed">
-        <origin xyz="0 0 ${ 0.5 - total_height/2}" rpy="0 0 0"/>
+        <origin xyz="0 0 ${0.4 - total_height/2}" rpy="0 0 0"/>
         <parent link="payload_link"/>
         <child link="pole_link"/>
@@ -95,9 +95,14 @@
             <parent link="payload_link"/>
             <child link="${laser_frame}"/>
-            <origin xyz="0.075 0 0.035" rpy="0 3.1415 0.0"/>
+            <xacro:if value="$(arg is_sim)">
+                <origin xyz="0.075 0 -0.01" rpy="0.0 0.0 3.1415"/>
+            </xacro:if>
+            <xacro:unless value="$(arg is_sim)">
+                <origin xyz="0.075 0 0.0" rpy="0 3.1415 0.0"/>
+            </xacro:unless>
         </joint>
         <link name="${laser_frame}">
             <visual>
-                <origin xyz="0 0 0" rpy="-1.57 3.1415 3.1415"/>
+                <origin xyz="0 0 0" rpy="-1.57 0.0 3.1415"/> <!-- rpy="-1.57 0.0 3.1415" real rover-->
                 <geometry>
                     <mesh filename="file://$(find rover_description_pkg)/meshes/rplidar_s2.dae"/>
@@ -105,5 +110,5 @@
             </visual>
             <collision>
-                <origin xyz="0 0 -0.05" rpy="0 0 3.1415"/>
+                <origin xyz="0 0 0" rpy="0 0 3.1415"/>
                 <geometry>
                     <cylinder radius="0.04" length="0.15"/>
@@ -116,4 +121,5 @@
             <topic>${laser_topic}</topic>
             <ignition_frame_id>rover/lidar_link</ignition_frame_id>
+            <gz_frame_id>rover/lidar_link</gz_frame_id>
             <update_rate>30</update_rate>
             <lidar>

Commit message: new rover simulation branch!

File: src/pkg/rover_description_pkg/urdf/rover.xacro (robot description, xacro)
@@ -8,7 +8,5 @@
 </link>
 <xacro:rover_base_frame parent_link="base_footprint"/>
-<!-- <xacro:rover_turret parent_link="rover_turret_plate"/> -->
 <!-- if it is in simulation -->
-<xacro:if value="$(arg is_sim)">
     <xacro:rover_wheels_sim left_joint="diff_drive_l_joint" right_joint="diff_drive_r_joint"/>
     <xacro:gazebo_diff_drive_controller left_joint="diff_drive_l_joint" right_joint="diff_drive_r_joint"/>
@@ -16,9 +14,3 @@
     <xacro:lidar_gazebo_sensor laser_frame="lidar_link" laser_topic="scan"/>
     <xacro:camera_gazebo camera_base_frame="camera_link" camera_topic="camera" camera_info_topic="camera_info"/>
-</xacro:if>
-<!-- if it is not in simulation -->
-<xacro:unless value="$(arg is_sim)">
-    <xacro:rover_rplidar_s1 laser_frame="laser"/>
-    <!-- <xacro:rover_camera_realsense_d435i camera_base_frame="camera_frame"/> -->
-</xacro:unless>
 </robot>

File: src/pkg/rover_description_pkg/urdf/rover_gazebo.xacro (robot description, xacro)
@@ -1,7 +1,4 @@
 <?xml version="1.0"?>
 <robot xmlns:xacro="http://www.ros.org/wiki/xacro" name="rover_gazebo">
-    <gazebo reference="chassis_link">
-        <material>Gazebo/DarkGrey</material>
-    </gazebo>
 <xacro:macro name="rover_wheels_sim" params="left_joint right_joint">
     <link name="fr_wheel_link">
@@ -137,5 +134,4 @@
   <joint name="camera_rgb_joint" type="fixed">
     <origin xyz="0.005 0.018 0.013" rpy="0 0 0"/>
-    <!-- <origin xyz="${r200_cam_rgb_px} ${r200_cam_rgb_py} ${r200_cam_rgb_pz}" rpy="0 0 0"/> -->
     <parent link="${camera_base_frame}"/>
     <child link="camera_rgb_frame"/>
@@ -150,5 +146,4 @@
   <joint name="camera_depth_joint" type="fixed">
     <origin xyz="0.005 0.028 0.013" rpy="0 0 0"/>
-    <!-- <origin xyz="${r200_cam_rgb_px} ${r200_cam_rgb_py + r200_cam_depth_offset} ${r200_cam_rgb_pz}" rpy="0 0 0"/> -->
     <parent link="${camera_base_frame}"/>
     <child link="camera_depth_frame"/>
@@ -156,5 +151,4 @@
   <link name="camera_depth_frame"/>
   <joint name="camera_depth_optical_joint" type="fixed">
-    <!-- <origin xyz="0 0 0" rpy="-1.57 0 -1.57"/> -->
     <origin xyz="0 0 0" rpy="0 0 0"/>
     <parent link="camera_depth_frame"/>

File: src/pkg/rover_description_pkg/urdf/rover_macro.xacro (robot description, xacro)
@@ -18,12 +18,10 @@
     <!-- Robot Parameters -->
     <xacro:property name="wheel_z_offset" value="0.020" />
-    <xacro:property name="wheel_x_offset" value="${wheel_axes_distance/2}" /> <!-- <xacro:property name="wheel_x_offset" value="0.145" /> -->
+    <xacro:property name="wheel_x_offset" value="${wheel_axes_distance/2}" />
     <xacro:property name="front_flipper_x_offset" value="-0.0035" />
-    <xacro:property name="wheel_y_offset" value="${(total_width-track_width)/2}" /> <!-- <xacro:property name="wheel_y_offset" value="0.18" /> -->
+    <xacro:property name="wheel_y_offset" value="${(total_width-track_width)/2}" />
     <xacro:property name="track_y_offset" value="0.11" />
     <xacro:property name="wheel_mass" value="1.25" />
     <xacro:property name="payload_z_offset" value="0.096" />
-    <!-- <xacro:include filename="$(find rover_description_pkg)/urdf/rover_dev_payload.urdf" />
-    <xacro:include filename="$(find rover_description_pkg)/urdf/rplidar_s2.urdf" /> -->
     <xacro:include filename="$(find rover_description_pkg)/urdf/imu.urdf" />
     <xacro:macro name="rover_base_frame" params="parent_link">
@@ -66,10 +64,4 @@
     </xacro:macro>
     <link name="payload_link">
-        <!-- <visual>
-            <origin xyz="0 0.0115 0" rpy="1.57 -0 1.57" />
-            <geometry>
-                <mesh filename="file://$(find roverrobotics_description)/meshes/rover_payload.dae"/>
-            </geometry>
-        </visual> -->
         <collision>
             <origin xyz="-0.1 0.0 0.04" rpy="0 0 0" />
@@ -98,14 +90,9 @@
             <parent link="payload_link"/>
             <child link="${laser_frame}"/>
-            <xacro:if value="$(arg is_sim)">
-                <origin xyz="0.075 0 -0.01" rpy="0.0 0.0 3.1415"/>
-            </xacro:if>
-            <xacro:unless value="$(arg is_sim)">
-                <origin xyz="0.075 0 0.0" rpy="0 3.1415 0.0"/>
-            </xacro:unless>
+            <origin xyz="0.075 0 -0.01" rpy="0.0 0.0 3.1415"/>
         </joint>
         <link name="${laser_frame}">
             <visual>
-                <origin xyz="0 0 0" rpy="-1.57 0.0 3.1415"/> <!-- rpy="-1.57 0.0 3.1415" real rover-->
+                <origin xyz="0 0 0" rpy="-1.57 0.0 3.1415"/>
                 <geometry>
                     <mesh filename="file://$(find rover_description_pkg)/meshes/rplidar_s2.dae"/>
@@ -156,17 +143,3 @@
     </gazebo> -->
     </xacro:macro>
-<!--
-    <xacro:macro name="rover_camera_realsense_d435i" params="camera_base_frame">
-        <xacro:include filename="$(find realsense2_description)/urdf/_d435i.urdf.xacro"/>
-        <xacro:sensor_d435i parent="${camera_base_frame}" use_nominal_extrinsics="true">
-            <origin xyz="0 0 0" rpy="0 0 0"/>
-        </xacro:sensor_d435i>
-        <joint name="rover_camera_joint" type="fixed">
-            <origin xyz="${chassis_length/2 - 0.02} 0.0 ${chassis_height - 0.01}" rpy="0.0 0.0 0.0"/>
-            <parent link="base_link"/>
-            <child link="${camera_base_frame}"/>
-        </joint>
-        <link name="${camera_base_frame}"/>
-    </xacro:macro>
--->
 </robot>
