Commit message: rover mesh changed and sensors positions adjust

File: src/pkg/rover_description_pkg/urdf/rover_gazebo.xacro (robot description, xacro)
@@ -117,5 +117,5 @@
     </xacro:sensor_d435i>  -->
     <joint name="camera_to_payload" type="fixed">
-        <origin xyz="0.02 0 ${1 -0.1 - total_height}" rpy="0 0 0"/>
+        <origin xyz="0.02 0 ${1 -0.129 - total_height}" rpy="0 0 0"/>
         <parent link="payload_link"/>
         <child link="${camera_base_frame}"/>

File: src/pkg/rover_description_pkg/urdf/rover_macro.xacro (robot description, xacro)
@@ -37,6 +37,9 @@
                 <origin xyz="0 0 -0.035" rpy="0 0 0" />
                 <geometry>
-                    <mesh filename="file://$(find rover_description_pkg)/meshes/prisma_rover.dae" scale="0.001 0.001 0.001"/>
+                    <mesh filename="file://$(find rover_description_pkg)/meshes/prisma_rover.stl" scale="0.001 0.001 0.001"/>
                 </geometry>
+                <material name="grey">
+                    <color rgba="0.2350821 0.2106182 0.2557221 1.0"/>
+                </material>
             </visual>
             <inertial>

Commit message: lidar 3d simulation

File: src/pkg/rover_description_pkg/urdf/rover_gazebo.xacro (robot description, xacro)
@@ -191,5 +191,5 @@
 			<pose>0 0.0175 0.5125 0 -0 0</pose>
 			<camera name="d435">
-                <point_cloud_topic>depth/color/points</point_cloud_topic>
+                <point_cloud_topic>depth/image_raw/points</point_cloud_topic>
                 <camera_info_topic>depth/camera_info</camera_info_topic>
 				<horizontal_fov>1.48702</horizontal_fov>
@@ -210,9 +210,87 @@
 		</sensor>
     </gazebo>
-    <gazebo>
+    <link name="livox_base">
+        <inertial>
+        <mass value="0.1"/>
+        <inertia ixx="0.01" ixy="0" ixz="0" iyy="0.01" iyz="0" izz="0.01"/>
+        </inertial>
+        <!-- <visual>
+        <origin rpy="0 0 0" xyz="0.00 0 0.0"/>
+        <geometry>
+            <mesh filename="package://gz_migration/meshes/livox_mid40.dae">
+            </mesh>
+        </geometry>
+        </visual> -->
+        <collision>
+            <origin xyz="0.075 0 0.15" rpy="0 0 0"/>
+            <geometry>
+                <cylinder radius="0.04" length="0.06"/>
+            </geometry>
+        </collision>
+    </link>
+    <link name="livox">
+        <inertial>
+        <mass value="0.1"/>
+        <inertia ixx="0.01" ixy="0" ixz="0" iyy="0.01" iyz="0" izz="0.01"/>
+        </inertial>
+    </link>
+    <joint name="base_link_to_livox" type="fixed">
+        <parent link="base_link"/>
+        <child link="livox_base"/>
+        <origin xyz="0.075 0 0.2" rpy="0 0 0"/>
+    </joint>
+    <joint name="livox_to_livox_base_joint" type="fixed">
+        <parent link="livox_base"/>
+        <child link="livox"/>
+        <origin rpy="0 0 0" xyz="0.0 0.0 0.0 "/>
+    </joint>
+    <gazebo reference="livox">
+        <sensor name="laser_livox" type="gpu_lidar">
+        <ignition_frame_id>rover/livox</ignition_frame_id>
+        <pose>0 0 0 0 0 0</pose>
+        <visualize>True</visualize>
+        <update_rate>10</update_rate>
+        <!-- This ray plgin is only for visualization. -->
+        <!--plugin filename="libros2_livox.so" name="livox_plugin"-->
+            <lidar>
+            <scan>
+                <horizontal>
+                    <samples>360</samples>
+                    <resolution>1</resolution>
+                    <min_angle>0</min_angle>
+                    <max_angle>6.28318</max_angle>
+                </horizontal>
+                <vertical>
+                    <samples>360</samples>
+                    <resolution>1</resolution>
+                    <min_angle>-0.12601266555555554</min_angle>
+                    <max_angle>0.9637699988888888</max_angle>
+                </vertical>
+            </scan>
+            <range>
+                <min>0.3</min>
+                <max>100.0</max>
+                <resolution>0.002</resolution>
+            </range>
+            <!-- <noise>
+                <type>gaussian</type>
+                <mean>0.0</mean>
+                <stddev>0.01</stddev>
+            </noise> -->
+            </lidar>
+            <!--visualize>False</visualize-->
+            <samples>24000</samples>
+            <downsample>1</downsample>
+            <csv_file_name>package://rover_description_pkg/scan_mode/mid360.csv</csv_file_name>
+            <!--ros_topic>${ros_topic}</ros_topic-->
+            <topic>/livox/scan</topic>
+        <!--/plugin-->
+        </sensor>
+    </gazebo>
+    <!-- <gazebo>
         <plugin filename="libignition-gazebo-sensors-system.so" name="ignition::gazebo::systems::Sensors">
             <render_engine>ogre2</render_engine>
         </plugin>
-    </gazebo>
+    </gazebo>     -->
 </xacro:macro>
     <!-- Gazebo Plugins -->
@@ -235,5 +313,5 @@
             <!-- Output -->
             <frame_id>rover/odom</frame_id>
-            <child_frame_id>rover/base_link</child_frame_id>
+            <child_frame_id>rover/base_footprint</child_frame_id>
             <!-- Topics -->
             <topic>/cmd_vel</topic>

File: src/pkg/rover_description_pkg/urdf/rover_macro.xacro (robot description, xacro)
@@ -137,9 +137,9 @@
         </sensor>
     </gazebo>
-    <!-- <gazebo>
+    <gazebo>
         <plugin filename="libignition-gazebo-sensors-system.so" name="ignition::gazebo::systems::Sensors">
             <render_engine>ogre2</render_engine>
         </plugin>
-    </gazebo> -->
+    </gazebo>
     </xacro:macro>
 </robot>

Commit message: pointcloud to laserscan, tentative of scan merge, navigation improved for silulation, leonardo arena gazebo fortress world

File: src/pkg/rover_description_pkg/urdf/rover_gazebo.xacro (robot description, xacro)
@@ -185,9 +185,9 @@
 		<sensor name="d435_depth" type="depth_camera">
 			<always_on>1</always_on>
-			<update_rate>10</update_rate>
+			<update_rate>30</update_rate>
 			<visualize>0</visualize>
 			<topic>depth/image_raw</topic>
             <ignition_frame_id>rover/camera_depth_optical_frame</ignition_frame_id>
-			<pose>0 0.0175 0.5125 0 -0 0</pose>
+			<pose>0 0.0 0.0 0 -0 0</pose>
 			<camera name="d435">
                 <point_cloud_topic>depth/image_raw/points</point_cloud_topic>
@@ -221,5 +221,5 @@
             </mesh>
         </geometry>
-        </visual> -->
+        </visual>
         <collision>
             <origin xyz="0.075 0 0.15" rpy="0 0 0"/>
@@ -227,5 +227,5 @@
                 <cylinder radius="0.04" length="0.06"/>
             </geometry>
-        </collision>
+        </collision> -->
     </link>
     <link name="livox">

Commit message: Simulation migrated to Garden + adjust for the usage of aruco detector and yolo

File: src/pkg/rover_description_pkg/urdf/rover_gazebo.xacro (robot description, xacro)
@@ -114,5 +114,5 @@
     </xacro:sensor_d435i>  -->
     <joint name="camera_to_payload" type="fixed">
-        <origin xyz="0.02 0 ${1 -0.129 - total_height}" rpy="0 0 0"/>
+        <origin xyz="0.1 0.0 0.04" rpy="0 0 0"/>
         <parent link="payload_link"/>
         <child link="${camera_base_frame}"/>
@@ -158,9 +158,9 @@
     <gazebo reference="${camera_base_frame}">
         <sensor name="d435_color" type="camera">
-            <topic>color/image_raw</topic>
+            <topic>rover/color/image_raw</topic>
             <ignition_frame_id>rover/camera_link</ignition_frame_id>
             <gz_frame_id>rover/camera_link</gz_frame_id>
             <camera name="d435">
-                <camera_info_topic>color/camera_info</camera_info_topic>
+                <camera_info_topic>rover/color/camera_info</camera_info_topic>
                 <horizontal_fov>1.21126</horizontal_fov>
 				<image>
@@ -187,10 +187,10 @@
 			<update_rate>30</update_rate>
 			<visualize>0</visualize>
-			<topic>depth/image_raw</topic>
+			<topic>rover/depth/image_raw</topic>
             <ignition_frame_id>rover/camera_depth_optical_frame</ignition_frame_id>
 			<pose>0 0.0 0.0 0 -0 0</pose>
 			<camera name="d435">
-                <point_cloud_topic>depth/image_raw/points</point_cloud_topic>
-                <camera_info_topic>depth/camera_info</camera_info_topic>
+                <point_cloud_topic>rover/depth/image_raw/points</point_cloud_topic>
+                <camera_info_topic>rover/depth/camera_info</camera_info_topic>
 				<horizontal_fov>1.48702</horizontal_fov>
 				<image>
@@ -245,5 +245,5 @@
         <origin rpy="0 0 0" xyz="0.0 0.0 0.0 "/>
     </joint>
-    <gazebo reference="livox">
+    <!-- <gazebo reference="livox">
         <sensor name="laser_livox" type="gpu_lidar">
         <ignition_frame_id>rover/livox</ignition_frame_id>
@@ -251,6 +251,5 @@
         <visualize>True</visualize>
         <update_rate>10</update_rate>
-        <!-- This ray plgin is only for visualization. -->
-        <!--plugin filename="libros2_livox.so" name="livox_plugin"-->
+        <plugin filename="libros2_livox.so" name="livox_plugin">
             <lidar>
             <scan>
@@ -273,19 +272,12 @@
                 <resolution>0.002</resolution>
             </range>
-            <!-- <noise>
-                <type>gaussian</type>
-                <mean>0.0</mean>
-                <stddev>0.01</stddev>
-            </noise> -->
             </lidar>
-            <!--visualize>False</visualize-->
             <samples>24000</samples>
             <downsample>1</downsample>
             <csv_file_name>package://rover_description_pkg/scan_mode/mid360.csv</csv_file_name>
-            <!--ros_topic>${ros_topic}</ros_topic-->
             <topic>/livox/scan</topic>
-        <!--/plugin-->
+        </plugin>
         </sensor>
-    </gazebo>
+    </gazebo> -->
     <!-- <gazebo>
         <plugin filename="libignition-gazebo-sensors-system.so" name="ignition::gazebo::systems::Sensors">
@@ -297,5 +289,6 @@
 <xacro:macro name="gazebo_diff_drive_controller" params="left_joint right_joint">
     <gazebo>
-        <plugin name="ignition::gazebo::systems::DiffDrive" filename="ignition-gazebo-diff-drive-system">
+        <!-- <plugin name="ignition::gazebo::systems::DiffDrive" filename="ignition-gazebo-diff-drive-system">  -->
+        <plugin name="gz::sim::systems::DiffDrive" filename="gz-sim-diff-drive-system">
             <num_wheel_pairs>2</num_wheel_pairs>
             <!-- Wheel Information -->
@@ -315,9 +308,10 @@
             <child_frame_id>rover/base_footprint</child_frame_id>
             <!-- Topics -->
-            <topic>/cmd_vel</topic>
+            <topic>/rover/cmd_vel</topic>
             <odom_topic>/odom/wheels</odom_topic>
-            <tf_topic>/tf_gazebo</tf_topic>
+            <!-- <tf_topic>/tf</tf_topic> -->
         </plugin>
-        <plugin filename="ignition-gazebo-joint-state-publisher-system" name="ignition::gazebo::systems::JointStatePublisher">
+        <!-- <plugin filename="ignition-gazebo-joint-state-publisher-system" name="ignition::gazebo::systems::JointStatePublisher"> -->
+        <plugin filename="gz-sim-joint-state-publisher-system" name="gz::sim::systems::JointStatePublisher">
             <topic>/joint_states</topic>
         </plugin>

File: src/pkg/rover_description_pkg/urdf/rover_macro.xacro (robot description, xacro)
@@ -90,5 +90,5 @@
             <parent link="payload_link"/>
             <child link="${laser_frame}"/>
-            <origin xyz="0.075 0 -0.01" rpy="0.0 0.0 3.1415"/>
+            <origin xyz="0.075 0 -0.01" rpy="0.0 0.0 0.0"/>
         </joint>
         <link name="${laser_frame}">
@@ -138,5 +138,6 @@
     </gazebo>
     <gazebo>
-        <plugin filename="libignition-gazebo-sensors-system.so" name="ignition::gazebo::systems::Sensors">
+        <!-- <plugin filename="libignition-gazebo-sensors-system.so" name="ignition::gazebo::systems::Sensors"> -->
+        <plugin filename="gz-sim-sensors-system" name="gz::sim::systems::Sensors">
             <render_engine>ogre2</render_engine>
         </plugin>
